File: SIradio/STM-SIradio.brd (EAGLE design)
At the start: 17.8 x 36 mm, 48 parts

Commit message: updated with v0.2 - see Readme for details
Parts:
- added LOGO1: OSHW-LOGOL, SparkFun-Aesthetics:OSHW-LOGO-L
Other:
- board text added: "20131205-01"
- board text added: "SIradio - Mini"

Commit message: few more tweaks
Routing:
- net GND: vias 59 -> 60
Changed lines of the file:
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@@
 <via x="12.065" y="35.08375" extent="1-16" drill="0.3302"/>
 <via x="10.795" y="33.81375" extent="1-16" drill="0.3302"/>
-<via x="8.89" y="26.3525" extent="1-16" drill="0.3302"/>
 <contactref element="U$3" pad="18"/>
 <contactref element="JP2" pad="1"/>
@@
 <via x="9.68375" y="16.98625" extent="1-16" drill="0.3302"/>
 <via x="10.31875" y="17.62125" extent="1-16" drill="0.3302"/>
+<via x="8.5725" y="26.19375" extent="1-16" drill="0.3302"/>
+<via x="9.2075" y="26.82875" extent="1-16" drill="0.3302"/>
 </signal>
 <signal name="3.3V">

Commit message: Updated with new VCXO footprint, seen readme for other specifics
Parts:
- FVXO-HC53BR-27: value OSCILLATORSMD6 -> (none); device SparkFun-FreqCtrl_TK:CRYSTAL-SMD-7.5X5.2-6PIN -> SparkFun-FreqCtrl:VCXO-SMD-5X3.2
- moved C38 9.75 mm to (8.10, 34.1)
- moved R22 1.27 mm to (8.10, 32.9)
- moved FVXO-HC53BR-27 0.57 mm to (8.26, 30.0)
Connections:
- net 3.3V: no longer FVXO-HC53BR-27.6INNER
- net GND: no longer FVXO-HC53BR-27.3INNER
- net N$1: no longer FVXO-HC53BR-27.1INNER
- net N$13: no longer FVXO-HC53BR-27.4INNER
- net TX_ENABLE: no longer FVXO-HC53BR-27.2INNER
Routing:
- net N$13: track 12.6 -> 10.1 mm
- net 3.3V: track 47.7 -> 45.6 mm
- net N$1: track 10.4 -> 8.36 mm
- net GND: track 3.13 -> 1.41 mm, vias 60 -> 67
