File: SIradio/STM-SIradio.brd (EAGLE design)
At the start: 17.8 x 36 mm, 49 parts

Commit message: First Version - PCB produced
Parts:
- C18: value 0.1uF -> 100nF
- C24: value 22pf -> 22pF
- moved C20 0.32 mm to (10.8, 23.8)
- moved R21 0.32 mm to (3.49, 29.5)
- moved C18 0.16 mm to (2.22, 31.8)
Connections:
- net GND: now also U$3.21; no longer U$3.GND
Changed lines of the file:
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@@
 <layer number="220" name="220bmp" color="21" fill="1" visible="no" active="no"/>
 <layer number="221" name="221bmp" color="22" fill="1" visible="no" active="no"/>
+<layer number="222" name="222bmp" color="23" fill="1" visible="no" active="no"/>
 <layer number="223" name="223bmp" color="24" fill="1" visible="no" active="no"/>
 <layer number="224" name="224bmp" color="25" fill="1" visible="no" active="no"/>
@@
 <attribute name="VALUE" x="14.478" y="17.399" size="0.4064" layer="27" font="vector" rot="R90"/>
 </element>
-<element name="C20" library="SparkFun-Capacitors" package="0603-CAP" value="470pF" x="10.795" y="23.495" smashed="yes">
-<attribute name="NAME" x="9.906" y="24.41575" size="0.4064" layer="25" font="vector"/>
-<attribute name="VALUE" x="9.779" y="22.352" size="0.4064" layer="27" font="vector"/>
+<element name="C20" library="SparkFun-Capacitors" package="0603-CAP" value="470pF" x="10.795" y="23.8125" smashed="yes">
+<attribute name="NAME" x="9.906" y="24.73325" size="0.4064" layer="25" font="vector"/>
+<attribute name="VALUE" x="9.779" y="22.6695" size="0.4064" layer="27" font="vector"/>
 </element>
 <element name="C21" library="SparkFun-Capacitors" package="0603-CAP" value="100nF" x="12.065" y="18.415" smashed="yes" rot="R90">
@@
 <attribute name="VALUE" x="5.969" y="4.572" size="0.4064" layer="27" font="vector"/>
 </element>
-<element name="C24" library="SparkFun-Capacitors" package="0603-CAP" value="22pf" x="4.7625" y="6.6675" smashed="yes" rot="R90">
+<element name="C24" library="SparkFun-Capacitors" package="0603-CAP" value="22pF" x="4.7625" y="6.6675" smashed="yes" rot="R90">
 <attribute name="NAME" x="3.20675" y="5.93725" size="0.4064" layer="25" font="vector" rot="R90"/>
 <attribute name="VALUE" x="5.9055" y="5.6515" size="0.4064" layer="27" font="vector" rot="R90"/>
@@
 <attribute name="VALUE" x="3.683" y="32.9565" size="0.4064" layer="27" font="vector" rot="R90"/>
 </element>
-<element name="C18" library="SparkFun-Capacitors" package="0603-CAP" value="0.1uF" x="2.2225" y="31.90875" smashed="yes">
-<attribute name="NAME" x="1.3335" y="30.607" size="0.4064" layer="25" font="vector"/>
-<attribute name="VALUE" x="1.2065" y="30.76575" size="0.4064" layer="27" font="vector"/>
+<element name="C18" library="SparkFun-Capacitors" package="0603-CAP" value="100nF" x="2.2225" y="31.75" smashed="yes">
+<attribute name="NAME" x="1.3335" y="30.44825" size="0.4064" layer="25" font="vector"/>
+<attribute name="VALUE" x="1.2065" y="30.607" size="0.4064" layer="27" font="vector"/>
 </element>
 <element name="C1" library="SparkFun-Capacitors" package="0603-CAP" value="56nF" x="1.27" y="33.9725" smashed="yes" rot="R90">
@@
 <attribute name="VALUE" x="4.953" y="32.9565" size="0.4064" layer="27" font="vector" rot="R90"/>
 </element>
-<element name="R21" library="SparkFun-Resistors" package="0603-RES" value="0" x="3.4925" y="29.845" smashed="yes" rot="R270">
-<attribute name="NAME" x="2.3495" y="29.62275" size="0.4064" layer="25" font="vector" rot="R270"/>
-<attribute name="VALUE" x="2.3495" y="30.861" size="0.4064" layer="27" font="vector" rot="R270"/>
+<element name="R21" library="SparkFun-Resistors" package="0603-RES" value="0" x="3.4925" y="29.5275" smashed="yes" rot="R270">
+<attribute name="NAME" x="2.3495" y="29.30525" size="0.4064" layer="25" font="vector" rot="R270"/>
+<attribute name="VALUE" x="2.3495" y="30.5435" size="0.4064" layer="27" font="vector" rot="R270"/>
 </element>
 <element name="R22" library="SparkFun-Resistors" package="0603-RES" value="10K" x="8.09625" y="32.86125" smashed="yes" rot="R180">
@@
 <via x="16.03375" y="18.7325" extent="1-16" drill="0.3302"/>
 <via x="16.8275" y="18.7325" extent="1-16" drill="0.3302"/>
-<contactref element="U$3" pad="GND"/>
+<contactref element="U$3" pad="21"/>
 <via x="7.9375" y="19.20875" extent="1-16" drill="0.3302"/>
 <via x="7.9375" y="20.47875" extent="1-16" drill="0.3302"/>
@@
 <wire x1="13.81125" y1="22.4125" x2="12.19625" y2="22.4125" width="0.4064" layer="1"/>
 <wire x1="12.19625" y1="22.4125" x2="12.065" y2="22.28125" width="0.6096" layer="1"/>
-<wire x1="12.065" y1="22.28125" x2="12.065" y2="23.075" width="0.4064" layer="1"/>
-<wire x1="12.065" y1="23.075" x2="11.645" y2="23.495" width="0.4064" layer="1"/>
 <wire x1="12.3825" y1="7.5175" x2="12.3825" y2="8.9925" width="0.8128" layer="1"/>
 <wire x1="12.3825" y1="8.9925" x2="13.17625" y2="9.78625" width="0.254" layer="1"/>
@@
 <wire x1="8.94625" y1="32.86125" x2="9.38" y2="32.4275" width="0.4064" layer="1"/>
 <wire x1="9.38" y1="32.4275" x2="9.38" y2="31.27375" width="0.4064" layer="1"/>
-<wire x1="11.645" y1="25.615" x2="11.645" y2="23.495" width="0.4064" layer="1"/>
 <wire x1="12.54125" y1="33.655" x2="10.63625" y2="33.655" width="0.4064" layer="16"/>
 <wire x1="10.63625" y1="33.655" x2="10.16" y2="34.13125" width="0.4064" layer="16"/>
+<wire x1="11.645" y1="25.615" x2="11.645" y2="23.8125" width="0.4064" layer="1"/>
+<wire x1="11.645" y1="23.8125" x2="11.645" y2="22.70125" width="0.4064" layer="1"/>
+<wire x1="11.645" y1="22.70125" x2="12.065" y2="22.28125" width="0.4064" layer="1"/>
 </signal>
 <signal name="N$18">
@@
 <contactref element="R21" pad="1"/>
 <wire x1="1.27" y1="33.1225" x2="2.54" y2="33.1225" width="0.4064" layer="1"/>
-<wire x1="2.54" y1="33.1225" x2="2.54" y2="32.44125" width="0.4064" layer="1"/>
-<wire x1="2.54" y1="32.44125" x2="3.0725" y2="31.90875" width="0.4064" layer="1"/>
-<wire x1="3.0725" y1="31.90875" x2="3.4925" y2="31.48875" width="0.4064" layer="1"/>
-<wire x1="3.4925" y1="31.48875" x2="3.4925" y2="30.695" width="0.4064" layer="1"/>
-<wire x1="3.4925" y1="30.695" x2="4.60375" y2="31.80625" width="0.4064" layer="1"/>
-<wire x1="4.60375" y1="31.80625" x2="4.7625" y2="31.80625" width="0.4064" layer="1"/>
+<wire x1="2.54" y1="33.1225" x2="2.54" y2="32.2825" width="0.4064" layer="1"/>
+<wire x1="2.54" y1="32.2825" x2="3.0725" y2="31.75" width="0.4064" layer="1"/>
+<wire x1="3.0725" y1="31.75" x2="3.4925" y2="31.33" width="0.4064" layer="1"/>
+<wire x1="3.4925" y1="31.33" x2="3.4925" y2="30.3775" width="0.4064" layer="1"/>
+<wire x1="4.7625" y1="31.80625" x2="4.7625" y2="31.75" width="0.4064" layer="1"/>
+<wire x1="4.7625" y1="31.75" x2="3.0725" y2="31.75" width="0.4064" layer="1"/>
 </signal>
 <signal name="MODULATION">
@@
 <wire x1="10.04875" y1="19.0975" x2="10.04875" y2="20.84375" width="0.254" layer="16"/>
 <wire x1="10.04875" y1="20.84375" x2="10.95375" y2="21.74875" width="0.254" layer="16"/>
-<wire x1="3.4925" y1="28.995" x2="3.4925" y2="28.2575" width="0.254" layer="1"/>
-<wire x1="3.4925" y1="28.2575" x2="3.01625" y2="27.78125" width="0.254" layer="1"/>
-<wire x1="3.01625" y1="27.78125" x2="3.01625" y2="19.20875" width="0.254" layer="1"/>
+<wire x1="3.01625" y1="28.20125" x2="3.01625" y2="19.20875" width="0.254" layer="1"/>
 <via x="3.01625" y="19.20875" extent="1-16" drill="0.3302"/>
 <wire x1="3.01625" y1="19.20875" x2="3.01625" y2="17.62125" width="0.254" layer="16"/>
@@
 <wire x1="4.60375" y1="17.30375" x2="3.33375" y2="17.30375" width="0.254" layer="1"/>
 <wire x1="3.33375" y1="17.30375" x2="3.01625" y2="17.62125" width="0.254" layer="1"/>
+<wire x1="3.01625" y1="28.20125" x2="3.4925" y2="28.6775" width="0.254" layer="1"/>
 </signal>
 <signal name="N$13">
